File: aps_passkey_hardware/aps_passkey_hardware.kicad_sch (KiCad schematic)
At the start: 0 parts

Commit message: schematic
Parts:
- added C1, C18, C2, C21, C3, C6: 4.7u, Capacitor_SMD:C_0402_1005Metric, symbol Device:C
- added C10, C11, C12, C13, C14, C15, C16, C17, C7, C8, C9: 100n, Capacitor_SMD:C_0402_1005Metric, symbol Device:C
- added C19, C20: 10u, Capacitor_SMD:C_0603_1608Metric, symbol Device:C
- added C4, C5: 33p, Capacitor_SMD:C_0402_1005Metric, symbol Device:C
- added D1: LED, LED_SMD:LED_0603_1608Metric, symbol Device:LED
- added J1: USB_A, user_imported_devices:USBPCB, symbol Connector:USB_A
- added L1: AOTA, easyeda2kicad:IND-SMD_L2.0-W1.6_AOTA-B201610S3R3-101-T, symbol easyeda2kicad:AOTA-B201610S3R3-101-T
- added R1: 33, Resistor_SMD:R_0402_1005Metric, symbol Device:R
- added R2, R3: 27R, Resistor_SMD:R_0402_1005Metric, symbol Device:R
- added R4, R5, R6: 1k, Resistor_SMD:R_0402_1005Metric, symbol Device:R
- added SW1: SW_Push, easyeda2kicad:SW-SMD_L3.9-W3.0-P4.45, symbol Switch:SW_Push
- added U1: RP2354A-QFN60, user_imported_devices:RP2350A_QFN-60_EP_7.75x7.75_Pitch0.4mm, symbol user_imported:RP2350A-QFN60
- added U2: TLV75512PDQNR, easyeda2kicad:X2SON-4_L1.0-W1.0-P0.65-TL-EP, symbol easyeda2kicad:TLV75512PDQNR
- added Y1: Crystal_GND24, Crystal:Crystal_SMD_3225-4Pin_3.2x2.5mm, symbol Device:Crystal_GND24
Connections:
- new net: L1.1, U1.48 (VREG_LX)
- new net: R5.2, U1.22 (XOUT)
- new net: D1.1 (K), R6.1
- new net: C20.1, C21.1, J1.1 (VBUS), U2.3 (EN), U2.4 (IN)
- new net: R4.1, SW1.2
- new net: C5.1, Y1.3
- new net: R3.1, U1.51 (USB_DM)
- new net: C4.1, Y1.1
- new net: C2.1, R1.2, U1.46 (VREG_AVDD)
- new net: D1.2 (A), U1.37 (GPIO25)
- new net: R2.1, U1.52 (USB_DP)
- new net +1V1: C1.1, C6.1, C7.1, C8.1, L1.2, U1.23 (DVDD), U1.39 (DVDD), U1.50 (VREG_FB), U1.6 (DVDD)
- new net +3V3: C10.1, C11.1, C12.1, C13.1, C14.1, C15.1, C16.1, C17.1, C18.1, C19.1, C3.1, C9.1, R1.1, U1.1 (IOVDD), U1.11 (IOVDD), U1.20 (IOVDD), U1.30 (IOVDD), U1.38 (IOVDD), U1.44 (ADC_AVDD), U1.45 (IOVDD), U1.49 (VREG_VIN), U1.53 (USB_OTP_VDD), U1.54 (QSPI_IOVDD), U2.1 (OUT)
- new net DM: J1.2 (D-), R3.2
- new net DP: J1.3 (D+), R2.2
- new net GND: C1.2, C10.2, C11.2, C12.2, C13.2, C14.2, C15.2, C16.2, C17.2, C18.2, C19.2, C2.2, C20.2, C21.2, C3.2, C4.2, C5.2, C6.2, C7.2, C8.2, C9.2, J1.4 (GND), J1.5 (Shield), R6.2, SW1.1, U1.47 (VREG_PGND), U1.61 (GND), U2.2 (GND), U2.5 (EP), Y1.2, Y1.4
- new net QSPI_SS: R4.2, U1.60 (QSPI_SS)
- new net XIN: U1.21 (XIN)
- new net XOUT: R5.1
- no-connect marks 0 -> 8

Commit message: new design
Parts:
- added U3: W25Q128JVS, Package_SO:SOIC-8_5.3x5.3mm_P1.27mm, symbol Memory_Flash:W25Q128JVS
Connections:
- net +3V3: now also U3.8 (VCC)
- net GND: now also U3.4 (GND)
- net QSPI_SS: now also U3.1 (~{CS})
- net XIN: now also C4.1, Y1.1
- net XOUT: now also C5.1, Y1.3
- net SD3: now reaches U1.55 (QSPI_SD3)
- net SD3: now also U3.7 (~{HOLD}/~{RESET}/IO_{3})
- net QSPI_SCLK: now reaches U1.56 (QSPI_SCLK)
- net QSPI_SCLK: now also U3.6 (CLK)
- net SD0: now reaches U1.57 (QSPI_SD0)
- net SD0: now also U3.5 (DI/IO_{0})
- net SD2: now reaches U1.58 (QSPI_SD2)
- net SD2: now also U3.3 (~{WP}/IO_{2})
- net SD1: now reaches U1.59 (QSPI_SD1)
- net SD1: now also U3.2 (DO/IO_{1})
- no-connect marks 8 -> 3
Other:
- moved on the sheet: R4, SW1

Commit message: New Design
Parts:
- U1: value RP2354A-QFN60 -> RP2350A-QFN60
Connections:
- net TR-: now reaches R3.1, U1.51 (USB_DM)
- net TR+: now reaches R2.1, U1.52 (USB_DP)
- net DM renamed D-
- net DP renamed D+
Changed lines of the file:
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@@
 		)
 	)
-	(global_label "DM"
+	(global_label "D-"
 		(shape input)
 		(at 233.68 53.34 0)
@@
 		)
 		(property "Intersheetrefs" "${INTERSHEET_REFS}"
-			(at 239.3866 53.34 0)
+			(at 239.5076 53.34 0)
 			(effects
 				(font
@@
 		)
 	)
-	(global_label "DP"
+	(global_label "D+"
 		(shape input)
 		(at 233.68 50.8 0)
@@
 		)
 		(property "Intersheetrefs" "${INTERSHEET_REFS}"
-			(at 239.2052 50.8 0)
+			(at 239.5076 50.8 0)
 			(effects
 				(font
@@
 		)
 	)
-	(global_label "DP"
+	(global_label "D+"
 		(shape input)
 		(at 33.02 41.91 0)
@@
 		)
 		(property "Intersheetrefs" "${INTERSHEET_REFS}"
-			(at 38.5452 41.91 0)
+			(at 38.8476 41.91 0)
 			(effects
 				(font
@@
 		)
 	)
-	(global_label "DM"
+	(global_label "D-"
 		(shape input)
 		(at 33.02 44.45 0)
@@
 		)
 		(property "Intersheetrefs" "${INTERSHEET_REFS}"
-			(at 38.7266 44.45 0)
-			(effects
-				(font
-					(size 1.27 1.27)
-				)
-				(justify left)
-				(hide yes)
-			)
+			(at 38.8476 44.45 0)
+			(effects
+				(font
+					(size 1.27 1.27)
+				)
+				(justify left)
+				(hide yes)
+			)
+		)
+	)
+	(hierarchical_label "TR+"
+		(shape input)
+		(at 223.52 50.8 90)
+		(effects
+			(font
+				(size 1.27 1.27)
+			)
+			(justify left)
+		)
+	)
+	(hierarchical_label "TR-"
+		(shape input)
+		(at 223.52 53.34 270)
+		(effects
+			(font
+				(size 1.27 1.27)
+			)
+			(justify right)
 		)
 	)
@@
 			)
 		)
-		(property "Value" "RP2354A-QFN60"
+		(property "Value" "RP2350A-QFN60"
 			(at 195.1833 148.59 0)
 			(effects

Commit message: pcb
Parts:
- removed U3: W25Q128JVS, Package_SO:SOIC-8_5.3x5.3mm_P1.27mm, symbol Memory_Flash:W25Q128JVS

Commit message: PCB Done
Connections:
- net at U1.15 (GPIO11): now also D1.2 (A)
- net at U1.37 (GPIO25): no longer D1.2 (A)
Other:
- moved on the sheet: D1, R6
Changed lines of the file:
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@@
 	(wire
 		(pts
+			(xy 223.52 91.44) (xy 233.68 91.44)
+		)
+		(stroke
+			(width 0)
+			(type default)
+		)
+	)
+	(wire
+		(pts
 			(xy 162.56 24.13) (xy 167.64 24.13)
 		)
@@
 	(wire
 		(pts
-			(xy 223.52 127) (xy 233.68 127)
-		)
-		(stroke
-			(width 0)
-			(type default)
-		)
-	)
-	(wire
-		(pts
 			(xy 204.47 44.45) (xy 208.28 44.45)
 		)
@@
 	(wire
 		(pts
-			(xy 241.3 127) (xy 246.38 127)
+			(xy 241.3 91.44) (xy 246.38 91.44)
 		)
 		(stroke
@@
 	(wire
 		(pts
-			(xy 254 127) (xy 256.54 127)
+			(xy 254 91.44) (xy 256.54 91.44)
 		)
 		(stroke
@@
 	(wire
 		(pts
-			(xy 256.54 127) (xy 256.54 128.27)
+			(xy 256.54 91.44) (xy 256.54 92.71)
 		)
 		(stroke
@@
 	(symbol
 		(lib_id "Device:R")
-		(at 250.19 127 90)
+		(at 250.19 91.44 90)
 		(unit 1)
 		(exclude_from_sim no)
@@
 		(dnp no)
 		(property "Reference" "R6"
-			(at 250.19 124.46 90)
+			(at 250.19 88.9 90)
 			(effects
 				(font
@@
 		)
 		(property "Value" "1k"
-			(at 250.19 127 90)
+			(at 250.19 91.44 90)
 			(effects
 				(font
@@
 		)
 		(property "Footprint" "Resistor_SMD:R_0402_1005Metric"
-			(at 250.19 128.778 90)
+			(at 250.19 93.218 90)
 			(effects
 				(font
@@
 		)
 		(property "Datasheet" "~"
-			(at 250.19 127 0)
+			(at 250.19 91.44 0)
 			(effects
 				(font
@@
 		)
 		(property "Description" "Resistor"
-			(at 250.19 127 0)
+			(at 250.19 91.44 0)
 			(effects
 				(font
@@
 	(symbol
 		(lib_id "Device:LED")
-		(at 237.49 127 180)
+		(at 237.49 91.44 180)
 		(unit 1)
 		(exclude_from_sim no)
@@
 		(fields_autoplaced yes)
 		(property "Reference" "D1"
-			(at 239.0775 119.38 0)
+			(at 239.0775 83.82 0)
 			(effects
 				(font
@@
 		)
 		(property "Value" "LED"
-			(at 239.0775 121.92 0)
+			(at 239.0775 86.36 0)
 			(effects
 				(font
@@
 		)
 		(property "Footprint" "LED_SMD:LED_0603_1608Metric"
-			(at 237.49 127 0)
+			(at 237.49 91.44 0)
 			(effects
 				(font
@@
 		)
 		(property "Datasheet" "~"
-			(at 237.49 127 0)
+			(at 237.49 91.44 0)
 			(effects
 				(font
@@
 		)
 		(property "Description" "Light emitting diode"
-			(at 237.49 127 0)
+			(at 237.49 91.44 0)
 			(effects
 				(font
@@
 		)
 		(property "Sim.Pins" "1=K 2=A"
-			(at 237.49 127 0)
+			(at 237.49 91.44 0)
 			(effects
 				(font
@@
 	(symbol
 		(lib_id "power:GND")
-		(at 256.54 128.27 0)
+		(at 256.54 92.71 0)
 		(unit 1)
 		(exclude_from_sim no)
@@
 		(dnp no)
 		(property "Reference" "#PWR017"
-			(at 256.54 134.62 0)
+			(at 256.54 99.06 0)
 			(effects
 				(font
@@
 		)
 		(property "Value" "GND"
-			(at 256.54 132.08 0)
+			(at 256.54 96.52 0)
 			(effects
 				(font
@@
 		)
 		(property "Footprint" ""
-			(at 256.54 128.27 0)
+			(at 256.54 92.71 0)
 			(effects
 				(font
@@
 		)
 		(property "Datasheet" ""
-			(at 256.54 128.27 0)
+			(at 256.54 92.71 0)
 			(effects
 				(font
@@
 		)
 		(property "Description" "Power symbol creates a global label with name \"GND\" , ground"
-			(at 256.54 128.27 0)
+			(at 256.54 92.71 0)
 			(effects
 				(font
